Commit message: added husky robot

File: general_description/robots/robot.urdf.xacro (robot description, xacro)
@@ -1,6 +1,13 @@
 <?xml version="1.0" ?>
 <robot xmlns:xacro="http://www.ros.org/wiki/xacro" name="general">
-    <xacro:include filename="$(find general_description)/config/config.urdf.xacro" />
+    <xacro:include filename="$(find general_description)/config/$(arg robot_name)_config.urdf.xacro" />
+    <xacro:include filename="$(find general_description)/urdf/material.urdf.xacro" />
     <xacro:include filename="$(find general_description)/urdf/inertia.urdf.xacro" />
     <xacro:include filename="$(find general_description)/urdf/chasis.urdf.xacro" />
+    <xacro:include filename="$(find general_description)/urdf/wheel.urdf.xacro" />
+    <!-- Adding four wheels -->
+    <xacro:wheel link_name="front_left_wheel" wheel_pos="${front_left_wheel_pos}" mesh_filename="${wheel_meshfile}"/>
+    <xacro:wheel link_name="front_right_wheel" wheel_pos="${front_right_wheel_pos}" mesh_filename="${wheel_meshfile}"/>
+    <xacro:wheel link_name="rear_left_wheel" wheel_pos="${rear_left_wheel_pos}" mesh_filename="${wheel_meshfile}"/>
+    <xacro:wheel link_name="rear_right_wheel" wheel_pos="${rear_right_wheel_pos}" mesh_filename="${wheel_meshfile}"/>
 </robot>

File: general_description/urdf/chasis.urdf.xacro (robot description, xacro)
@@ -2,5 +2,5 @@
 <robot xmlns:xacro="http://www.ros.org/wiki/xacro">
     <!-- Setting up base_link -->
-    <link name="${chasis_link_name}">
+    <link name="base_link">
         <origin rpy="0 0 0" xyz="0 0 0"/>
         <collision>
@@ -18,19 +18,19 @@
         </visual>
     </link>
-    <!-- chasis_link_name_inertia have the inertia details -->
-    <link name="${chasis_link_name}_inertia">
+    <!-- base_link_inertia have the inertia details -->
+    <link name="base_link_inertia">
         <xacro:inertia_box m="${chasis_mass}" x="${chasis_length}" y="${chasis_width}" z="${chasis_height}" xyz="0 0 0"/>
     </link>
-    <joint name="${chasis_link_name}_inertial_joint" type="fixed">
+    <joint name="base_link_inertial_joint" type="fixed">
         <origin xyz="0 0 ${chasis_height/2}" rpy="0 0 0" />
-        <parent link="${chasis_link_name}" />
-        <child link="${chasis_link_name}_inertia" />
+        <parent link="base_link" />
+        <child link="base_link_inertia" />
     </joint>
     <!-- Footprint link on the ground -->
     <link name="footprint" />
     <joint name="footprint_joint" type="fixed">
-        <origin xyz="0 0 ${wheel_radius - (wheel_center_to_chasis_center - chasis_height/2)}" rpy="0 0 0" />
+        <origin xyz="0 0 ${wheel_center_to_chasis_center + wheel_radius - chasis_height/2}" rpy="0 0 0" />
         <parent link="footprint" />
-        <child link="${chasis_link_name}" />
+        <child link="base_link" />
     </joint>
 </robot>

File: general_description/urdf/material.urdf.xacro (robot description, xacro)
@@ -2,5 +2,5 @@
 <robot xmlns:xacro="http://www.ros.org/wiki/xacro">
 	<material name="wheel">
-		<color rgba="0 0 1 1.0"/>
+		<color rgba="0 1.0 1.0 1.0"/>
 	</material>
 	<material name="chasis">
