Commit message: gazebo control

File: general_description/config/husky_config.urdf.xacro (robot description, xacro)
@@ -15,10 +15,13 @@
     <xacro:property name="wheel_radius" value="0.178" />
     <xacro:property name="wheel_thickness" value="0.114" />
-    <xacro:property name="wheel_meshfile" value="${robot_name}/wheel.dae" />
+    <xacro:property name="left_wheel_meshfile" value="${robot_name}/wheel.dae" />
+    <xacro:property name="right_wheel_meshfile" value="${robot_name}/wheel.dae" />
     <!-- Add the height of the wheel wrt to center of the chasis instead of the numeric value -->
     <xacro:property name="z_pos_wheel" value="${-wheel_center_to_chasis_center + chasis_height/2}" />
-    <xacro:property name="front_left_wheel_pos" value="-0.256 -0.2854 ${z_pos_wheel}" />
-    <xacro:property name="front_right_wheel_pos" value="-0.256 0.2854 ${z_pos_wheel}" />
-    <xacro:property name="rear_left_wheel_pos" value="0.256 -0.2854 ${z_pos_wheel}" />
-    <xacro:property name="rear_right_wheel_pos" value="0.256 0.2854 ${z_pos_wheel}" />
+    <xacro:property name="x_pos_wheel" value="0.256" />
+    <xacro:property name="y_pos_wheel" value="0.2854" />
+    <xacro:property name="front_left_wheel_pos" value="${x_pos_wheel} ${y_pos_wheel} ${z_pos_wheel}" />
+    <xacro:property name="front_right_wheel_pos" value="${x_pos_wheel} ${-y_pos_wheel} ${z_pos_wheel}" />
+    <xacro:property name="rear_left_wheel_pos" value="${-x_pos_wheel} ${y_pos_wheel} ${z_pos_wheel}" />
+    <xacro:property name="rear_right_wheel_pos" value="${-x_pos_wheel} -${y_pos_wheel} ${z_pos_wheel}" />
 </robot>

File: general_description/config/pioneer3at_config.urdf.xacro (robot description, xacro)
@@ -13,11 +13,14 @@
     <xacro:property name="wheel_radius" value="0.111" />
     <xacro:property name="wheel_thickness" value="0.096" />
-    <xacro:property name="wheel_meshfile" value="${robot_name}/wheel.dae" />
+    <xacro:property name="left_wheel_meshfile" value="${robot_name}/left_wheel.dae" />
+    <xacro:property name="right_wheel_meshfile" value="${robot_name}/right_wheel.dae" />
     <!-- Absolute value of height of wheel center from the center of the chasis -->
     <xacro:property name="wheel_center_to_chasis_center" value="0.066" />
     <xacro:property name="z_pos_wheel" value="${-wheel_center_to_chasis_center + chasis_height/2}" />
-    <xacro:property name="front_left_wheel_pos" value="-0.134 -0.199 ${z_pos_wheel}" />
-    <xacro:property name="front_right_wheel_pos" value="-0.134 0.199 ${z_pos_wheel}" />
-    <xacro:property name="rear_left_wheel_pos" value="0.134 -0.199 ${z_pos_wheel}" />
-    <xacro:property name="rear_right_wheel_pos" value="0.134 0.199 ${z_pos_wheel}" />
+    <xacro:property name="x_pos_wheel" value="0.134" />
+    <xacro:property name="y_pos_wheel" value="0.199" />
+    <xacro:property name="front_left_wheel_pos" value="${x_pos_wheel} ${y_pos_wheel} ${z_pos_wheel}" />
+    <xacro:property name="front_right_wheel_pos" value="${x_pos_wheel} ${-y_pos_wheel} ${z_pos_wheel}" />
+    <xacro:property name="rear_left_wheel_pos" value="${-x_pos_wheel} ${y_pos_wheel} ${z_pos_wheel}" />
+    <xacro:property name="rear_right_wheel_pos" value="${-x_pos_wheel} -${y_pos_wheel} ${z_pos_wheel}" />
 </robot>

File: general_description/robots/robot.urdf.xacro (robot description, xacro)
@@ -6,8 +6,9 @@
     <xacro:include filename="$(find general_description)/urdf/chasis.urdf.xacro" />
     <xacro:include filename="$(find general_description)/urdf/wheel.urdf.xacro" />
+    <xacro:include filename="$(find general_description)/urdf/gazebo.xacro" />
     <!-- Adding four wheels -->
-    <xacro:wheel link_name="front_left_wheel" wheel_pos="${front_left_wheel_pos}" mesh_filename="${wheel_meshfile}"/>
-    <xacro:wheel link_name="front_right_wheel" wheel_pos="${front_right_wheel_pos}" mesh_filename="${wheel_meshfile}"/>
-    <xacro:wheel link_name="rear_left_wheel" wheel_pos="${rear_left_wheel_pos}" mesh_filename="${wheel_meshfile}"/>
-    <xacro:wheel link_name="rear_right_wheel" wheel_pos="${rear_right_wheel_pos}" mesh_filename="${wheel_meshfile}"/>
+    <xacro:wheel link_name="front_left_wheel" wheel_pos="${front_left_wheel_pos}" mesh_filename="${left_wheel_meshfile}"/>
+    <xacro:wheel link_name="front_right_wheel" wheel_pos="${front_right_wheel_pos}" mesh_filename="${left_wheel_meshfile}"/>
+    <xacro:wheel link_name="rear_left_wheel" wheel_pos="${rear_left_wheel_pos}" mesh_filename="${left_wheel_meshfile}"/>
+    <xacro:wheel link_name="rear_right_wheel" wheel_pos="${rear_right_wheel_pos}" mesh_filename="${left_wheel_meshfile}"/>
 </robot>

File: general_description/urdf/wheel.urdf.xacro (robot description, xacro)
@@ -38,6 +38,6 @@
 		</transmission>
     <gazebo reference="${link_name}" >
-      <mu1 value="100.0" />
-      <mu2 value="100.0" />
+      <mu1 value="1.0" />
+      <mu2 value="1.0" />
       <kp  value="100000.0" />
       <kd  value="1.0" />

Commit message: added lidar plugin

File: general_description/config/husky_config.urdf.xacro (robot description, xacro)
@@ -18,10 +18,14 @@
     <xacro:property name="right_wheel_meshfile" value="${robot_name}/wheel.dae" />
     <!-- Add the height of the wheel wrt to center of the chasis instead of the numeric value -->
-    <xacro:property name="z_pos_wheel" value="${-wheel_center_to_chasis_center + chasis_height/2}" />
     <xacro:property name="x_pos_wheel" value="0.256" />
     <xacro:property name="y_pos_wheel" value="0.2854" />
-    <xacro:property name="front_left_wheel_pos" value="${x_pos_wheel} ${y_pos_wheel} ${z_pos_wheel}" />
-    <xacro:property name="front_right_wheel_pos" value="${x_pos_wheel} ${-y_pos_wheel} ${z_pos_wheel}" />
-    <xacro:property name="rear_left_wheel_pos" value="${-x_pos_wheel} ${y_pos_wheel} ${z_pos_wheel}" />
-    <xacro:property name="rear_right_wheel_pos" value="${-x_pos_wheel} -${y_pos_wheel} ${z_pos_wheel}" />
+    <!-- Lidar Addition and position of sensor wrt -->
+    <xacro:arg name="enable_lidar" default="true"/>
+        <xacro:property name="lidar_link_name" value="front_lidar" />
+        <xacro:property name="lidar_xyz" value="-0.15 0 0.354" />
+        <xacro:property name="lidar_rpy" value="0 0 0" />
+        <xacro:property name="min_scan_angle" value="-3.14" />
+        <xacro:property name="max_scan_angle" value="3.14" />
+        <xacro:property name="min_scan_range" value="0.5" />
+        <xacro:property name="max_scan_range" value="20" />
 </robot>

File: general_description/config/pioneer3at_config.urdf.xacro (robot description, xacro)
@@ -17,10 +17,15 @@
     <!-- Absolute value of height of wheel center from the center of the chasis -->
     <xacro:property name="wheel_center_to_chasis_center" value="0.066" />
-    <xacro:property name="z_pos_wheel" value="${-wheel_center_to_chasis_center + chasis_height/2}" />
     <xacro:property name="x_pos_wheel" value="0.134" />
     <xacro:property name="y_pos_wheel" value="0.199" />
-    <xacro:property name="front_left_wheel_pos" value="${x_pos_wheel} ${y_pos_wheel} ${z_pos_wheel}" />
-    <xacro:property name="front_right_wheel_pos" value="${x_pos_wheel} ${-y_pos_wheel} ${z_pos_wheel}" />
-    <xacro:property name="rear_left_wheel_pos" value="${-x_pos_wheel} ${y_pos_wheel} ${z_pos_wheel}" />
-    <xacro:property name="rear_right_wheel_pos" value="${-x_pos_wheel} -${y_pos_wheel} ${z_pos_wheel}" />
+    <!-- Sensor Addition to the platform -->
+    <!-- Lidar Addition -->
+    <xacro:arg name="enable_lidar" default="true"/>
+        <xacro:property name="lidar_link_name" value="front_lidar" />
+        <xacro:property name="lidar_xyz" value="0 0 0.3" />
+        <xacro:property name="lidar_rpy" value="0 0 0" />
+        <xacro:property name="min_scan_angle" value="-3.14" />
+        <xacro:property name="max_scan_angle" value="3.14" />
+        <xacro:property name="min_scan_range" value="0.5" />
+        <xacro:property name="max_scan_range" value="20" />
 </robot>

File: general_description/robots/robot.urdf.xacro (robot description, xacro)
@@ -6,5 +6,11 @@
     <xacro:include filename="$(find general_description)/urdf/chasis.urdf.xacro" />
     <xacro:include filename="$(find general_description)/urdf/wheel.urdf.xacro" />
+    <xacro:include filename="$(find general_description)/urdf/sensor.urdf.xacro" />
     <xacro:include filename="$(find general_description)/urdf/gazebo.xacro" />
+    <xacro:property name="z_pos_wheel" value="${-wheel_center_to_chasis_center + chasis_height/2}" />
+    <xacro:property name="front_left_wheel_pos" value="${x_pos_wheel} ${y_pos_wheel} ${z_pos_wheel}" />
+    <xacro:property name="front_right_wheel_pos" value="${x_pos_wheel} ${-y_pos_wheel} ${z_pos_wheel}" />
+    <xacro:property name="rear_left_wheel_pos" value="${-x_pos_wheel} ${y_pos_wheel} ${z_pos_wheel}" />
+    <xacro:property name="rear_right_wheel_pos" value="${-x_pos_wheel} -${y_pos_wheel} ${z_pos_wheel}" />
     <!-- Adding four wheels -->
     <xacro:wheel link_name="front_left_wheel" wheel_pos="${front_left_wheel_pos}" mesh_filename="${left_wheel_meshfile}"/>
@@ -12,3 +18,7 @@
     <xacro:wheel link_name="rear_left_wheel" wheel_pos="${rear_left_wheel_pos}" mesh_filename="${left_wheel_meshfile}"/>
     <xacro:wheel link_name="rear_right_wheel" wheel_pos="${rear_right_wheel_pos}" mesh_filename="${left_wheel_meshfile}"/>
+    <!-- Adding sensors -->
+    <xacro:if value="$(arg enable_lidar)">
+        <xacro:sensor_lidar link_name="${lidar_link_name}" xyz="${lidar_xyz}" rpy="${lidar_rpy}"/>
+    </xacro:if>
 </robot>

File: general_description/urdf/gazebo.xacro (robot description, xacro)
@@ -9,3 +9,36 @@
     </plugin>
   </gazebo>
+  <xacro:if value="$(arg enable_lidar)">
+    <gazebo reference="${lidar_link_name}">
+      <sensor type="ray" name="${lidar_link_name}">
+          <pose>0 0 0 0 0 0</pose>
+          <visualize>true</visualize>
+          <update_rate>25</update_rate>
+          <ray>
+              <scan>
+                  <horizontal>
+                      <samples>720</samples>
+                      <resolution>0.25</resolution>
+                      <min_angle>${min_scan_angle}</min_angle>
+                      <max_angle>${max_scan_angle}</max_angle>
+                  </horizontal>
+              </scan>
+              <range>
+                  <min>${min_scan_range}</min>
+                  <max>${max_scan_range}</max>
+                  <resolution>0.25</resolution>
+              </range>
+              <noise>
+                  <type>gaussian</type>
+                  <mean>0.0</mean>
+                  <stddev>0.01</stddev>
+              </noise>
+          </ray>
+          <plugin name="gazebo_ros_head_hokuyo_controller" filename="libgazebo_ros_laser.so">
+              <topicName>${lidar_link_name}_scan</topicName>
+              <frameName>${lidar_link_name}</frameName>
+          </plugin>
+      </sensor>
+    </gazebo>
+  </xacro:if>
 </robot>

File: general_description/urdf/material.urdf.xacro (robot description, xacro)
@@ -7,3 +7,6 @@
 		<color rgba="0 1 0 1.0"/>
 	</material>
+	<material name="lidar">
+		<color rgba="1 0 0 1.0"/>
+	</material>
 </robot>
