Commit message: stereo and gps

File: general_description/config/husky_config.urdf.xacro (robot description, xacro)
@@ -8,20 +8,21 @@
     <xacro:property name="chasis_width" value="0.571" />
     <xacro:property name="chasis_height" value="0.249" />
-    <xacro:property name="chasis_meshfile" value="${robot_name}/chasis.dae" />
     <!-- Wheel configuration -->
-    <!-- Absolute value of distance of wheel center from the center of the chasis -->
-    <xacro:property name="wheel_center_to_chasis_center" value="0.092" />
     <xacro:property name="wheel_mass" value="2" />
     <xacro:property name="wheel_radius" value="0.178" />
     <xacro:property name="wheel_thickness" value="0.114" />
-    <xacro:property name="left_wheel_meshfile" value="${robot_name}/wheel.dae" />
-    <xacro:property name="right_wheel_meshfile" value="${robot_name}/wheel.dae" />
-    <!-- Add the height of the wheel wrt to center of the chasis instead of the numeric value -->
+    <!-- Absolute value of height of wheel center from the center of the chasis -->
+    <xacro:property name="wheel_center_to_chasis_center" value="0.092" />
     <xacro:property name="x_pos_wheel" value="0.256" />
     <xacro:property name="y_pos_wheel" value="0.2854" />
-    <!-- Lidar Addition and position of sensor wrt -->
+    <!-- Sensor Addition to the platform -->
+    <!-- All the position of sensor is wrt the center of the chasis -->
+    <!-- Lidar Addition -->
     <xacro:arg name="enable_lidar" default="true"/>
         <xacro:property name="lidar_link_name" value="front_lidar" />
-        <xacro:property name="lidar_xyz" value="-0.15 0 0.354" />
+        <xacro:property name="visualize_scan" value="false" />
+        <xacro:property name="x_pos_lidar" value="-0.15" />
+        <xacro:property name="y_pos_lidar" value="0" />
+        <xacro:property name="z_pos_lidar" value="0.229" />
         <xacro:property name="lidar_rpy" value="0 0 0" />
         <xacro:property name="min_scan_angle" value="-3.14" />
@@ -29,3 +30,31 @@
         <xacro:property name="min_scan_range" value="0.5" />
         <xacro:property name="max_scan_range" value="20" />
+    <!-- IMU sensor Addition -->
+    <xacro:arg name="enable_imu" default="true"/>
+        <xacro:property name="imu_link_name" value="imu_link" />
+        <xacro:property name="x_pos_imu" value="0.19" />
+        <xacro:property name="y_pos_imu" value="0" />
+        <xacro:property name="z_pos_imu" value="0.149" />
+        <xacro:property name="imu_rpy" value="0 -1.57 3.1416" />
+    <!-- Stereo Camera Addition -->
+    <xacro:arg name="enable_stereo" default="true"/>
+        <xacro:property name="camera_link_name" value="camera_link" />
+        <xacro:property name="min_camera_range" value="0.1" />
+        <xacro:property name="max_camera_range" value="8.0" />
+        <xacro:property name="camera_fps" value="30" />
+        <xacro:property name="camera_width" value="640" />
+        <xacro:property name="camera_height" value="480" />
+        <xacro:property name="camera_h_fov" value="1.5184351666" />
+        <xacro:property name="camera_v_fov" value="1.01229011" />
+        <xacro:property name="x_pos_camera" value="0.26" />
+        <xacro:property name="y_pos_camera" value="0" />
+        <xacro:property name="z_pos_camera" value="0.125" />
+        <xacro:property name="camera_rpy" value="0 0 0" />
+    <!-- GPS Sensor Addition -->
+    <xacro:arg name="enable_gps" default="true"/>
+        <xacro:property name="gps_link_name" value="gps_link" />
+        <xacro:property name="x_pos_gps" value="0" />
+        <xacro:property name="y_pos_gps" value="0" />
+        <xacro:property name="z_pos_gps" value="0" />
+        <xacro:property name="gps_rpy" value="0 0 0" />
 </robot>

File: general_description/config/pioneer3at_config.urdf.xacro (robot description, xacro)
@@ -8,11 +8,8 @@
     <xacro:property name="chasis_width" value="0.383" />
     <xacro:property name="chasis_height" value="0.195" />
-    <xacro:property name="chasis_meshfile" value="${robot_name}/chasis.dae" />
     <!-- Wheel configuration -->
     <xacro:property name="wheel_mass" value="2" />
     <xacro:property name="wheel_radius" value="0.111" />
     <xacro:property name="wheel_thickness" value="0.096" />
-    <xacro:property name="left_wheel_meshfile" value="${robot_name}/left_wheel.dae" />
-    <xacro:property name="right_wheel_meshfile" value="${robot_name}/right_wheel.dae" />
     <!-- Absolute value of height of wheel center from the center of the chasis -->
     <xacro:property name="wheel_center_to_chasis_center" value="0.066" />
@@ -20,8 +17,12 @@
     <xacro:property name="y_pos_wheel" value="0.199" />
     <!-- Sensor Addition to the platform -->
+    <!-- All the position of sensor is wrt the center of the chasis -->
     <!-- Lidar Addition -->
     <xacro:arg name="enable_lidar" default="true"/>
         <xacro:property name="lidar_link_name" value="front_lidar" />
-        <xacro:property name="lidar_xyz" value="0 0 0.3" />
+        <xacro:property name="visualize_scan" value="false" />
+        <xacro:property name="x_pos_lidar" value="0" />
+        <xacro:property name="y_pos_lidar" value="0" />
+        <xacro:property name="z_pos_lidar" value="0.202" />
         <xacro:property name="lidar_rpy" value="0 0 0" />
         <xacro:property name="min_scan_angle" value="-3.14" />
@@ -29,3 +30,31 @@
         <xacro:property name="min_scan_range" value="0.5" />
         <xacro:property name="max_scan_range" value="20" />
+    <!-- IMU sensor Addition -->
+    <xacro:arg name="enable_imu" default="true"/>
+        <xacro:property name="imu_link_name" value="imu_link" />
+        <xacro:property name="x_pos_imu" value="0" />
+        <xacro:property name="y_pos_imu" value="0" />
+        <xacro:property name="z_pos_imu" value="0.12" />
+        <xacro:property name="imu_rpy" value="0 -1.57 3.1416" />
+    <!-- Stereo Camera Addition -->
+    <xacro:arg name="enable_stereo" default="true"/>
+        <xacro:property name="camera_link_name" value="camera_link" />
+        <xacro:property name="min_camera_range" value="0.1" />
+        <xacro:property name="max_camera_range" value="8.0" />
+        <xacro:property name="camera_fps" value="30" />
+        <xacro:property name="camera_width" value="640" />
+        <xacro:property name="camera_height" value="480" />
+        <xacro:property name="camera_h_fov" value="1.5184351666" />
+        <xacro:property name="camera_v_fov" value="1.01229011" />
+        <xacro:property name="x_pos_camera" value="0.25" />
+        <xacro:property name="y_pos_camera" value="0" />
+        <xacro:property name="z_pos_camera" value="0.098" />
+        <xacro:property name="camera_rpy" value="0 0 0" />
+    <!-- GPS Sensor Addition -->
+    <xacro:arg name="enable_gps" default="true"/>
+        <xacro:property name="gps_link_name" value="gps_link" />
+        <xacro:property name="x_pos_gps" value="0" />
+        <xacro:property name="y_pos_gps" value="0" />
+        <xacro:property name="z_pos_gps" value="0" />
+        <xacro:property name="gps_rpy" value="0 0 0" />
 </robot>

File: general_description/robots/robot.urdf.xacro (robot description, xacro)
@@ -14,11 +14,24 @@
     <xacro:property name="rear_right_wheel_pos" value="${-x_pos_wheel} -${y_pos_wheel} ${z_pos_wheel}" />
     <!-- Adding four wheels -->
-    <xacro:wheel link_name="front_left_wheel" wheel_pos="${front_left_wheel_pos}" mesh_filename="${left_wheel_meshfile}"/>
-    <xacro:wheel link_name="front_right_wheel" wheel_pos="${front_right_wheel_pos}" mesh_filename="${left_wheel_meshfile}"/>
-    <xacro:wheel link_name="rear_left_wheel" wheel_pos="${rear_left_wheel_pos}" mesh_filename="${left_wheel_meshfile}"/>
-    <xacro:wheel link_name="rear_right_wheel" wheel_pos="${rear_right_wheel_pos}" mesh_filename="${left_wheel_meshfile}"/>
+    <xacro:wheel link_name="front_left_wheel" wheel_pos="${front_left_wheel_pos}" mesh_filename="${robot_name}/left_wheel.dae"/>
+    <xacro:wheel link_name="front_right_wheel" wheel_pos="${front_right_wheel_pos}" mesh_filename="${robot_name}/right_wheel.dae"/>
+    <xacro:wheel link_name="rear_left_wheel" wheel_pos="${rear_left_wheel_pos}" mesh_filename="${robot_name}/left_wheel.dae"/>
+    <xacro:wheel link_name="rear_right_wheel" wheel_pos="${rear_right_wheel_pos}" mesh_filename="${robot_name}/right_wheel.dae"/>
     <!-- Adding sensors -->
+    <!-- Lidar Sensor -->
     <xacro:if value="$(arg enable_lidar)">
-        <xacro:sensor_lidar link_name="${lidar_link_name}" xyz="${lidar_xyz}" rpy="${lidar_rpy}"/>
+        <xacro:sensor_lidar link_name="${lidar_link_name}" xyz="${x_pos_lidar} ${y_pos_lidar} ${z_pos_lidar + chasis_height/2}" rpy="${lidar_rpy}"/>
+    </xacro:if>
+    <!-- IMU Sensor -->
+    <xacro:if value="$(arg enable_imu)">
+        <xacro:sensor_imu link_name="${imu_link_name}" xyz="${x_pos_imu} ${y_pos_imu} ${z_pos_imu + chasis_height/2}" rpy="${imu_rpy}"/>
+    </xacro:if>
+    <!-- Stereo Camera Sensor -->
+    <xacro:if value="$(arg enable_stereo)">
+        <xacro:sensor_stereo link_name="${camera_link_name}" xyz="${x_pos_camera} ${y_pos_camera} ${z_pos_camera + chasis_height/2}" rpy="${camera_rpy}"/>
+    </xacro:if>
+    <!-- GPS Sensor -->
+    <xacro:if value="$(arg enable_gps)">
+        <xacro:sensor_gps link_name="${gps_link_name}" xyz="${x_pos_gps} ${y_pos_gps} ${y_pos_gps + chasis_height/2}" rpy="${gps_rpy}"/>
     </xacro:if>
 </robot>

File: general_description/urdf/chasis.urdf.xacro (robot description, xacro)
@@ -13,5 +13,5 @@
             <origin rpy="0 0 0" xyz="0 0 ${chasis_height/2}"/>
             <geometry>
-            <mesh filename="package://general_description/meshes/${chasis_meshfile}" scale="1 1 1"/>
+            <mesh filename="package://general_description/meshes/${robot_name}/chasis.dae" scale="1 1 1"/>
             </geometry>
             <material name="chasis"/>

File: general_description/urdf/gazebo.xacro (robot description, xacro)
@@ -5,4 +5,5 @@
     <plugin name="gazebo_ros_control" filename="libgazebo_ros_control.so">
       <robotNamespace>$(arg robot_name)</robotNamespace>
+      <robotParam>$(arg robot_name)_description</robotParam>
       <robotSimType>gazebo_ros_control/DefaultRobotHWSim</robotSimType>
       <legacyModeNS>true</legacyModeNS>
@@ -13,5 +14,5 @@
       <sensor type="ray" name="${lidar_link_name}">
           <pose>0 0 0 0 0 0</pose>
-          <visualize>true</visualize>
+          <visualize>${visualize_scan}</visualize>
           <update_rate>25</update_rate>
           <ray>
@@ -36,5 +37,6 @@
           </ray>
           <plugin name="gazebo_ros_head_hokuyo_controller" filename="libgazebo_ros_laser.so">
-              <topicName>${lidar_link_name}_scan</topicName>
+              <robotNamespace>$(arg robot_name)</robotNamespace>
+              <topicName>scan</topicName>
               <frameName>${lidar_link_name}</frameName>
           </plugin>
@@ -42,3 +44,92 @@
     </gazebo>
   </xacro:if>
+  <xacro:if value="$(arg enable_lidar)">
+    <gazebo reference="${imu_link_name}">
+      <gravity>true</gravity>
+      <sensor name="imu_sensor" type="imu">
+        <always_on>true</always_on>
+        <update_rate>100</update_rate>
+        <visualize>true</visualize>
+        <topic>__default_topic__</topic>
+        <plugin filename="libgazebo_ros_imu_sensor.so" name="imu_plugin">
+          <robotNamespace>$(arg robot_name)</robotNamespace>
+          <topicName>imu</topicName>
+          <bodyName>${imu_link_name}</bodyName>
+          <updateRateHZ>10.0</updateRateHZ>
+          <gaussianNoise>0.0</gaussianNoise>
+          <xyzOffset>0 0 0</xyzOffset>
+          <rpyOffset>0 0 0</rpyOffset>
+          <frameName>${imu_link_name}</frameName>
+          <initialOrientationAsReference>false</initialOrientationAsReference>
+        </plugin>
+        <pose>0 0 0 0 0 0</pose>
+      </sensor>
+    </gazebo>
+  </xacro:if>
+  <xacro:if value="$(arg enable_stereo)">
+    <gazebo reference="${camera_link_name}">
+      <turnGravityOff>true</turnGravityOff>
+      <sensor type="depth" name="camera_realsense_depth">
+        <update_rate>${camera_fps}</update_rate>
+        <camera>
+          <!-- 75x65 degree FOV for the depth sensor -->
+          <horizontal_fov>${camera_h_fov}</horizontal_fov>
+          <vertical_fov>${camera_v_fov}</vertical_fov>
+          <image>
+            <width>${camera_width}</width>
+            <height>${camera_height}</height>
+            <!-- TODO: check what format the Realsense hardware delivers and set this to match! -->
+            <format>RGB8</format>
+          </image>
+          <clip>
+            <!-- give the color sensor a maximum range of 50m so that the simulation renders nicely -->
+            <near>0.01</near>
+            <far>50.0</far>
+          </clip>
+        </camera>
+        <plugin name="kinect_controller" filename="libgazebo_ros_openni_kinect.so">
+          <robotNamespace>$(arg robot_name)</robotNamespace>
+          <baseline>0.2</baseline>
+          <alwaysOn>true</alwaysOn>
+          <updateRate>${camera_fps}</updateRate>
+          <cameraName>realsense</cameraName>
+          <imageTopicName>color/image_raw</imageTopicName>
+          <cameraInfoTopicName>color/camera_info</cameraInfoTopicName>
+          <depthImageTopicName>depth/image_rect_raw</depthImageTopicName>
+          <depthImageInfoTopicName>depth/camera_info</depthImageInfoTopicName>
+          <pointCloudTopicName>depth/color/points</pointCloudTopicName>
+          <frameName>${camera_link_name}_gazebo</frameName>
+          <pointCloudCutoff>${min_camera_range}</pointCloudCutoff>
+          <pointCloudCutoffMax>${max_camera_range}</pointCloudCutoffMax>
+          <distortionK1>0.00000001</distortionK1>
+          <distortionK2>0.00000001</distortionK2>
+          <distortionK3>0.00000001</distortionK3>
+          <distortionT1>0.00000001</distortionT1>
+          <distortionT2>0.00000001</distortionT2>
+          <CxPrime>0</CxPrime>
+          <Cx>0</Cx>
+          <Cy>0</Cy>
+          <focalLength>0</focalLength>
+          <hackBaseline>0</hackBaseline>
+        </plugin>
+      </sensor>
+    </gazebo>
+  </xacro:if>
+  <xacro:if value="$(arg enable_gps)">
+    <gazebo>
+      <plugin name="gps_controller" filename="libhector_gazebo_ros_gps.so">
+        <robotNamespace>$(arg robot_name)</robotNamespace>
+        <updateRate>40</updateRate>
+        <bodyName>${gps_link_name}</bodyName>
+        <frameId>${gps_link_name}</frameId>
+        <topicName>navsat/fix</topicName>
+        <velocityTopicName>navsat/vel</velocityTopicName>
+        <referenceLatitude>49.9</referenceLatitude>
+        <referenceLongitude>8.9</referenceLongitude>
+        <referenceHeading>0</referenceHeading>
+        <referenceAltitude>0</referenceAltitude>
+        <drift>0.0001 0.0001 0.0001</drift>
+      </plugin>
+    </gazebo>
+  </xacro:if>
 </robot>

File: general_description/urdf/material.urdf.xacro (robot description, xacro)
@@ -10,3 +10,6 @@
 		<color rgba="1 0 0 1.0"/>
 	</material>
+	<material name="camera">
+		<color rgba="0.74 0.74 0.74 1.0"/>
+	</material>
 </robot>

File: general_description/urdf/sensor.urdf.xacro (robot description, xacro)
@@ -26,16 +26,63 @@
     </joint>
     </xacro:macro>
-  <!-- <xacro:macro name="zed_sensor" params="name"> -->
-    <!-- All the below links and joints are according to zed manual details -->
-    <!-- Links which are to be attached as child with ${name} -->
-    <!-- <link name="${name}_left_frame" />
-    <link name="${name}_left_optical_frame"/>
-    <link name="${name}_right_frame" />
-    <link name="${name}_right_optical_frame"/> -->
-    <!-- Joints to attach these links with the zed_front -->
-    <!-- <xacro:joint_sensor name="${name}_left_joint" parent="${name}" child="${name}_left_frame" origin_xyz="0 0.06 0" origin_rpy="0 0 0"/>
-    <xacro:joint_sensor name="${name}_left_optical_joint" parent="${name}_left_frame" child="${name}_left_optical_frame" origin_xyz="0 0 0" origin_rpy="-1.57079632679 0.0 -1.57079632679"/>
-    <xacro:joint_sensor name="${name}_right_joint" parent="${name}" child="${name}_right_frame" origin_xyz="0 -0.06 0" origin_rpy="0 0 0"/>
-    <xacro:joint_sensor name="${name}_right_optical_joint" parent="${name}_right_frame" child="${name}_right_optical_frame" origin_xyz="0 0 0" origin_rpy="-1.57079632679 0.0 -1.57079632679"/>
-  </xacro:macro> -->
+  <!-- Adding macro for IMU -->
+  <xacro:macro name="sensor_imu" params="link_name xyz rpy">
+    <link name="${link_name}"/>
+  <!-- IMU joint -->
+    <joint name="${link_name}_joint" type="fixed">
+      <origin rpy="${rpy}" xyz="${xyz}"/>
+      <child link="${link_name}"/>
+      <parent link="base_link"/>
+    </joint>
+  </xacro:macro>
+  <!-- Adding macro for Stereo Camera -->
+  <xacro:macro name="sensor_stereo" params="link_name xyz rpy">
+      <!-- this link is the origin for the camera's data -->
+    <link name="${link_name}" />
+      <!--
+        The gazebo plugin aligns the depth data with the Z axis, with X=left and Y=up
+        ROS expects the depth data along the X axis, with Y=left and Z=up
+        This link only exists to give the gazebo plugin the correctly-oriented frame
+      -->
+    <link name="${link_name}_gazebo" />
+      <joint name="${link_name}_gazebo_joint" type="fixed">
+        <parent link="${link_name}"/>
+        <child link="${link_name}_gazebo"/>
+        <origin xyz="0.0 0 0" rpy="-1.5707963267948966 0 -1.5707963267948966"/>
+      </joint>
+    <link name="${link_name}_realsense_lens">
+      <visual>
+        <!--
+          the model's origin is in the middle & it's rotated to lie in
+          the optical standard with X left, Y up, and Z forward
+        -->
+        <origin xyz="-0.0115 0 0.0100" rpy="1.570796 0 -1.570796" />
+        <geometry>
+          <!-- Origin of this mesh is the base of the bracket. -->
+          <mesh filename="package://general_description/meshes/sensors/d415.stl" />
+        </geometry>
+        <material name="camera" />
+      </visual>
+    </link>
+    <joint type="fixed" name="${link_name}_realsense_lens_joint">
+      <origin xyz="${xyz}" rpy="${rpy}" />
+      <parent link="base_link" />
+      <child link="${link_name}_realsense_lens" />
+    </joint>
+    <joint type="fixed" name="${link_name}_realsense_joint">
+      <origin xyz="0.025 0 0" rpy="0 0 0" />
+      <parent link="${link_name}_realsense_lens" />
+      <child link="${link_name}" />
+    </joint>
+  </xacro:macro>
+    <!-- Adding macro for GPS -->
+  <xacro:macro name="sensor_gps" params="link_name xyz rpy">
+    <link name="${link_name}"/>
+  <!-- IMU joint -->
+    <joint name="${link_name}_joint" type="fixed">
+      <origin rpy="${rpy}" xyz="${xyz}"/>
+      <child link="${link_name}"/>
+      <parent link="base_link"/>
+    </joint>
+  </xacro:macro>
 </robot>
