Commit message: segbot added

File: general_description/config/segbot_config.urdf.xacro (robot description, xacro)
@@ -2,18 +2,18 @@
 <robot xmlns:xacro="http://www.ros.org/wiki/xacro">
     <!-- Robot Name -->
-    <xacro:property name="robot_name" value="husky" />
+    <xacro:property name="robot_name" value="segbot" />
     <!-- Chasis configuration -->
     <xacro:property name="chasis_mass" value="5" />
-    <xacro:property name="chasis_length" value="0.985" />
-    <xacro:property name="chasis_width" value="0.571" />
-    <xacro:property name="chasis_height" value="0.249" />
+    <xacro:property name="chasis_length" value="0.991" />
+    <xacro:property name="chasis_width" value="0.596" />
+    <xacro:property name="chasis_height" value="0.331" />
     <!-- Wheel configuration -->
     <xacro:property name="wheel_mass" value="2" />
-    <xacro:property name="wheel_radius" value="0.178" />
-    <xacro:property name="wheel_thickness" value="0.114" />
+    <xacro:property name="wheel_radius" value="0.2665" />
+    <xacro:property name="wheel_thickness" value="0.169" />
     <!-- Absolute value of height of wheel center from the center of the chasis -->
-    <xacro:property name="wheel_center_to_chasis_center" value="0.092" />
-    <xacro:property name="x_pos_wheel" value="0.256" />
-    <xacro:property name="y_pos_wheel" value="0.2854" />
+    <xacro:property name="wheel_center_to_chasis_center" value="-0.032" />
+    <xacro:property name="x_pos_wheel" value="0.2877" />
+    <xacro:property name="y_pos_wheel" value="0.3368" />
     <!-- Sensor Addition to the platform -->
     <!-- All the position of sensor is wrt the center of the chasis -->
@@ -24,5 +24,5 @@
         <xacro:property name="x_pos_lidar" value="0" />
         <xacro:property name="y_pos_lidar" value="0" />
-        <xacro:property name="z_pos_lidar" value="0.229" />
+        <xacro:property name="z_pos_lidar" value="0.26" />
         <xacro:property name="lidar_rpy" value="0 0 0" />
         <xacro:property name="min_scan_angle" value="-3.14" />
@@ -47,7 +47,7 @@
         <xacro:property name="camera_h_fov" value="1.5184351666" />
         <xacro:property name="camera_v_fov" value="1.01229011" />
-        <xacro:property name="x_pos_camera" value="0.26" />
+        <xacro:property name="x_pos_camera" value="0.45" />
         <xacro:property name="y_pos_camera" value="0" />
-        <xacro:property name="z_pos_camera" value="0.125" />
+        <xacro:property name="z_pos_camera" value="0.15" />
         <xacro:property name="camera_rpy" value="0 0 0" />
     <!-- GPS Sensor Addition -->
